Commit message: updated files

File: urdf_asm/urdf/urdf_asm.urdf (robot description, URDF)
Before this commit: robot urdf_asm, 9 links, 8 joints
Joints:
- joint Lower0: origin xyz=0.055094 0.0144 0 rpy=1.5708 -1.5708 0 -> xyz=0.0550943670538193 0.0144 0 rpy=1.57079632679489 -1.5707963267949 0
- joint Lower3: origin xyz=0.055094 0.0144 0 rpy=1.5708 -1.5708 0 -> xyz=0.0550943670538193 0.0144 0 rpy=1.57079632679491 -1.5707963267949 0
- joint Upper1: limit lower=0 upper=1.57 effort=0 velocity=0 -> lower=-1.57 upper=0 effort=0 velocity=0
- joint Upper2: origin xyz=-0.030849 -0.030849 0.001 rpy=1.5708 0 3.1416 -> xyz=-0.0308492424049169 -0.0308492424049181 0.000999999999999996 rpy=1.5707963267949 0 3.14159265358979
- joint Upper3: limit lower=0 upper=1.57 effort=0 velocity=0 -> lower=-1.57 upper=0 effort=0 velocity=0

Commit message: updated some stuff

File: urdf_asm/urdf/urdf_asm.urdf (robot description, URDF)
Before this commit: robot urdf_asm, 9 links, 8 joints
Links:
- link Lower0_Link: geometry collision mesh filename=../meshes/Lower0_Link.STL; visual mesh filename=../meshes/Lower0_Link.STL
- link Lower1_Link: geometry collision mesh filename=../meshes/Lower1_Link.STL; visual mesh filename=../meshes/Lower1_Link.STL
- link Lower2_Link: geometry collision mesh filename=../meshes/Lower2_Link.STL; visual mesh filename=../meshes/Lower2_Link.STL
- link Lower3_Link: geometry collision mesh filename=../meshes/Lower3_Link.STL; visual mesh filename=../meshes/Lower3_Link.STL
- link Upper0_Link: geometry collision mesh filename=../meshes/Upper0_Link.STL; visual mesh filename=../meshes/Upper0_Link.STL
- link Upper1_Link: geometry collision mesh filename=../meshes/Upper1_Link.STL; visual mesh filename=../meshes/Upper1_Link.STL
- link Upper2_Link: geometry collision mesh filename=../meshes/Upper2_Link.STL; visual mesh filename=../meshes/Upper2_Link.STL
- link Upper3_Link: geometry collision mesh filename=../meshes/Upper3_Link.STL; visual mesh filename=../meshes/Upper3_Link.STL
- link base_link: geometry collision mesh filename=../meshes/base_link.STL; visual mesh filename=../meshes/base_link.STL

Commit message: updated urdf

File: urdf_asm/urdf/urdf_asm.urdf (robot description, URDF)
Before this commit: robot urdf_asm, 9 links, 8 joints
Links:
- link Lower0_Link: mass 0.00418426133217533 -> 0.0041843; geometry collision mesh filename=package://urdf_asm/meshes/Lower0_Link.STL; visual mesh filename=package://urdf_asm/meshes/Lower0_Link.STL
- link Lower1_Link: mass 0.00418426133217533 -> 0.0041843; geometry collision mesh filename=package://urdf_asm/meshes/Lower1_Link.STL; visual mesh filename=package://urdf_asm/meshes/Lower1_Link.STL
- link Lower2_Link: mass 0.00418426133217533 -> 0.0041843; geometry collision mesh filename=package://urdf_asm/meshes/Lower2_Link.STL; visual mesh filename=package://urdf_asm/meshes/Lower2_Link.STL
- link Lower3_Link: mass 0.00418426133217533 -> 0.0041843; geometry collision mesh filename=package://urdf_asm/meshes/Lower3_Link.STL; visual mesh filename=package://urdf_asm/meshes/Lower3_Link.STL
- link Upper0_Link: mass 0.0118251186545954 -> 0.011825; geometry collision mesh filename=package://urdf_asm/meshes/Upper0_Link.STL; visual mesh filename=package://urdf_asm/meshes/Upper0_Link.STL
- link Upper1_Link: mass 0.0118251181300378 -> 0.04; geometry collision mesh filename=package://urdf_asm/meshes/Upper1_Link.STL; visual mesh filename=package://urdf_asm/meshes/Upper1_Link.STL
- link Upper2_Link: mass 0.0118251186545954 -> 0.04; geometry collision mesh filename=package://urdf_asm/meshes/Upper2_Link.STL; visual mesh filename=package://urdf_asm/meshes/Upper2_Link.STL
- link Upper3_Link: mass 0.0118251181300378 -> 0.04; geometry collision mesh filename=package://urdf_asm/meshes/Upper3_Link.STL; visual mesh filename=package://urdf_asm/meshes/Upper3_Link.STL
- link base_link: mass 0.0587031197951744 -> 0.16; geometry collision mesh filename=package://urdf_asm/meshes/base_link.STL; visual mesh filename=package://urdf_asm/meshes/base_link.STL
Joints:
- joint Lower0: limit (none) -> lower=-0.35 upper=0.8 effort=0.19 velocity=12; origin xyz=0.0550943670538193 0.0144 0 rpy=1.57079632679489 -1.5707963267949 0 -> xyz=0.055094 0.0144 0 rpy=1.5708 -1.5708 0; type continuous -> revolute
- joint Lower1: limit (none) -> lower=-0.35 upper=0.8 effort=0.19 velocity=12; origin xyz=0.0550943670538193 0.0144 0 rpy=1.57079632679489 -1.5707963267949 0 -> xyz=0.055094 0.0144 0 rpy=1.5708 -1.5708 0; type continuous -> revolute
- joint Lower2: limit (none) -> lower=-0.35 upper=0.8 effort=0.19 velocity=12; origin xyz=0.0550943670538193 0.0144 0 rpy=1.57079632679491 -1.5707963267949 0 -> xyz=0.055094 0.0144 0 rpy=1.5708 -1.5708 0; type continuous -> revolute
- joint Lower3: limit (none) -> lower=-0.35 upper=0.8 effort=0.19 velocity=12; origin xyz=0.0550943670538193 0.0144 0 rpy=1.57079632679491 -1.5707963267949 0 -> xyz=0.055094 0.0144 0 rpy=1.5708 -1.5708 0; type continuous -> revolute
- joint Upper0: limit lower=0 upper=1.57 effort=0 velocity=0 -> lower=0 upper=1.57 effort=0.19 velocity=12; type continuous -> revolute
- joint Upper1: limit lower=-1.57 upper=0 effort=0 velocity=0 -> lower=-1.57 upper=0 effort=0.19 velocity=12; type continuous -> revolute
- joint Upper2: limit lower=0 upper=1.57 effort=0 velocity=0 -> lower=0 upper=1.57 effort=0.19 velocity=12; origin xyz=-0.0308492424049169 -0.0308492424049181 0.000999999999999996 rpy=1.5707963267949 0 3.14159265358979 -> xyz=-0.030849 -0.030849 0.001 rpy=1.5708 0 3.1416; type continuous -> revolute
- joint Upper3: limit lower=-1.57 upper=0 effort=0 velocity=0 -> lower=-1.57 upper=0 effort=0.19 velocity=12; type continuous -> revolute

Commit message: added collision geometry

File: urdf_asm/urdf/urdf_asm.urdf (robot description, URDF)
Before this commit: robot urdf_asm, 9 links, 8 joints
Links:
- link Lower0_Link: geometry collision box size=0.01 0.01 0.08; visual mesh filename=../meshes/Lower0_Link.STL
- link Lower1_Link: geometry collision box size=0.01 0.01 0.08; visual mesh filename=../meshes/Lower1_Link.STL
- link Lower2_Link: geometry collision box size=0.01 0.01 0.08; visual mesh filename=../meshes/Lower2_Link.STL
- link Lower3_Link: geometry collision box size=0.01 0.01 0.08; visual mesh filename=../meshes/Lower3_Link.STL
- link Upper0_Link: geometry collision box size=0.05 0.013 0.013; visual mesh filename=../meshes/Upper0_Link.STL
- link Upper1_Link: geometry collision box size=0.05 0.013 0.013; visual mesh filename=../meshes/Upper1_Link.STL
- link Upper2_Link: geometry collision box size=0.05 0.013 0.013; visual mesh filename=../meshes/Upper2_Link.STL
- link Upper3_Link: geometry collision box size=0.05 0.013 0.013; visual mesh filename=../meshes/Upper3_Link.STL
- link base_link: geometry collision box size=0.07 0.07 0.02; visual mesh filename=../meshes/base_link.STL
